File: src/AQ_sensor_GSM.sch (EAGLE design)
At the start: 120 parts, among them IC1 MIC29302WU, J1 F-1X03-SIP-100-32, J3 PJ-002BH, Q1 MMBT2222, Q2 MMBT2222, Q3 MMBT2222, Q4 MMBT2222, Q5 MMBT2222, Q6 MMBT2222, Q7 MMBT2222, U3 TEXAS_INSTRUMENTS_LM1117IMP-3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, U5 TXS0108EPWR, X1 53048-08

Commit message: Routed
Parts:
- removed C22, C25, C26, C27, C5: ECA-1HM220, Resistor_Capacitor:ECA-1HM220
- removed C6: EEEFN1C471P, EEEFN1C471P:EEEFN1C471P
- removed C7: 100nf, 06035C104K4T2A:06035C104K4T2A
- removed CHARGE: PCM12SMTR, AQ_sensor_MRC:PCM12SMTR
- removed D5: ESD56151W04, 4.7V TVS Diode:1N4148WS_RR
- removed IC1: MIC29302WU, MIC29302WU:MIC29302WU
- removed LIPO/BUCK, USB/BATT: TL2285EE, TL2285EE:TL2285EE
- removed POWER: RED, led:LEDCHIP-LED0603
- removed Q1: MMBT2222, MMBT2222_:MMBT2222
- removed R10: 47K, rcl:R-EU_R0603
- removed R11: 470R, rcl:R-EU_R0603
- removed R9: 100k, rcl:R-EU_R0603
- removed SOLAR_IN: 10118192-0001LF, AQ_sensor_GSM:10118192-0001LF
- removed U$1: (no value), MT2492:MT2492MT2492
- removed X1: 53048-08, AQ_sensor_GSM:53048-08
- added 5V: 2828XX-2282834-2, Connector:2828XX-2282834-2
- added BATT, PWR: TL2285EE, TL2285EE:TL2285EE
- added CHARGER: KMR621NGLFS, AQ_sensor_GSM:KMR621NGLFS
- added D4, D6, D7: SS54-HF, SS54-HF schottkey Diode:SS54-HF
- added GPIO, PROG: PINHD-1X4, Connector:PINHD-1X4
- added J2: 53261-0871, 53261-0871:53261-0871
- added MT2492: MT2492, MT2492:MT2492MT2492
- added PO: RED, led:LEDCHIP-LED0603
- added PWR_ON: ORANGE, led:LEDCHIP-LED0603
- C2: value 470uf -> 100uF; device T495X477K010ATE100:T495X477K010ATE100 -> rcl:CPOL-EUD
- C3: value 100nf -> 100uF; device 06035C104K4T2A:06035C104K4T2A -> rcl:CPOL-EUD
- R2: value 51K -> 1k; device rcl:R-EU_R0603 -> SparkFun-Resistors:1.20KOHM-0603-1/10W-1%
- R3: value 4.7K -> 47k; device rcl:R-EU_R0603 -> SparkFun-Resistors:1.20KOHM-0603-1/10W-1%
- R8: value 47K -> 10k; device rcl:R-EU_R0603 -> SparkFun-Resistors:1.20KOHM-0603-1/10W-1%
- renumbered C_P to CHARGING
Connections:
- removed net +5V: R14.2, SV2.1, U3.IN, USB/BATT.COM1, USB/BATT.COM2, X1-8.S
- removed net 3.8V: C6.1, C7.2, D5.K, IC1.OUT, LIPO/BUCK.NC1, LIPO/BUCK.NC2, R11.2, R9.2
- removed net 4.2V: C29.1, L2.2, LIPO/BUCK.NO1, LIPO/BUCK.NO2, R19.2, U$2.BAT
- removed net BVIN: C5.1, J3.1, R7.2, SOLAR_IN.VUSB, U$1.VIN
- removed net D+: PB_IN.D+, SOLAR_IN.D+
- removed net D-: PB_IN.D-, SOLAR_IN.D-
- removed net N$36: Q1.B, R3.2
- removed net N$37: Q1.E, R8.2
- removed net N$38: IC1.ADJ, R10.2, R9.1
- removed net TF-CLK: SV2.7
- removed net TF-CS: SV2.9
- removed net TF-MISO: SV2.8
- removed net TF-MOSI: SV2.10
- new net 4.5-16V: C3.+, MT2492.VIN, PWR.COM1, PWR.COM2, R2.1, R7.2
- new net 5VT: D4.K, PWR.NO1, PWR.NO2
- new net BMSV: R3.2, R8.1, SV2.15
- new net G_ADC0: EC200_GSM.ADC0, GPIO.1
- new net G_ADC1: EC200_GSM.ADC1, GPIO.2
- new net G_ADC2: EC200_GSM.ADC2
- new net G_GPIO1: EC200_GSM.GPIO1
- new net G_I2C_SCL: EC200_GSM.I2C_SCL, GPIO.4
- new net G_I2C_SDA: EC200_GSM.I2C_SDA, GPIO.3
- new net G_SPI_CLK: EC200_GSM.SPI_CLK
- new net G_SPI_CS: EC200_GSM.SPI_CS
- new net G_SPI_MISO: EC200_GSM.SPI_MISO
- new net G_SPI_MOSI: EC200_GSM.SPI_MOSI
- new net G_USB_BOOT: EC200_GSM.USB_BOOT, PROG.1
- new net G_USB_D+: EC200_GSM.USB_DP, PB_IN.D+
- new net G_USB_D-: EC200_GSM.USB_DM, PB_IN.D-
- new net G_USB_VBUS: EC200_GSM.USB_VBUS
- new net LBV: BATT.COM1, BATT.COM2, LIPO.1, R3.1
- new net N$59: D4.A, PB_IN.VUSB
- new net N$60: D7.K, J3.2, J3.3
- new net N$61: D6.A, J3.1
- net 5V_IN: now also 5V.1; no longer C22.1
- net 5V_OUT: now also C2.+, J2.8, R14.2, SV2.1, U3.IN; no longer C25.1, C26.1, C27.1, USB/BATT.NO1, USB/BATT.NO2
- net GND: now also 5V.2, C2.-, C3.-, CHARGER.2, D7.A, J2.7, MT2492.GND, PO.C, PROG.4, PWR_ON.C, R8.2; no longer C2.2, C22.2, C25.2, C26.2, C27.2, C3.1, C5.2, C6.2, C7.1, CHARGE.2, D5.A, IC1.GND, J3.2, J3.3, POWER.C, R10.1, R11.1, R8.1, SOLAR_IN.GND, SOLAR_IN.ID, SOLAR_IN.SHIELD, U$1.GND, X1-7.S
- net MCU_RXD: now also PROG.2
- net MCU_TXD: now also PROG.3
- net N$10: now also MT2492.FB; no longer U$1.FB
- net N$11: now also MT2492.EN; no longer U$1.EN
- net N$20: now also CHARGER.1; no longer CHARGE.1
- net N$25: now also PO.A; no longer POWER.A
- net N$3: now also MT2492.BS; no longer U$1.BS
- net N$35: now also PWR_ON.A, R2.2; no longer IC1.EN, Q1.C, R2.1
- net N$6: now also MT2492.SW; no longer U$1.SW
- net PMS_RX: now also J2.5; no longer X1-5.S
- net PMS_TX: now also J2.4; no longer X1-4.S
- net VBAT_EN: no longer R3.1
- net VUSB: now also D6.K, PWR.NC1, PWR.NC2; no longer C2.1, C3.2, IC1.VIN, PB_IN.VUSB, R2.2, USB/BATT.NC1, USB/BATT.NC2
- net V_LIPO: now also BATT.NO1, BATT.NO2, C29.1, L2.2, R19.2, U$2.BAT; no longer LIPO.1, LIPO/BUCK.COM1, LIPO/BUCK.COM2
Other:
- note added: "GSM RESET"
- note removed: "POWER KEY"
- moved on the sheet: C14, C21, C8, J3, L1, LIPO, R1, R14, R6, R7, U3

Commit message: Routed - Minus DW01
Changed lines of the file:
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@@
 <part name="R14" library="rcl" library_urn="urn:adsk.eagle:library:334" deviceset="R-EU_" device="R0603" package3d_urn="urn:adsk.eagle:package:23555/3" value="1K"/>
 <part name="GND32" library="supply1" library_urn="urn:adsk.eagle:library:371" deviceset="GND" device=""/>
-<part name="P+1" library="supply1" library_urn="urn:adsk.eagle:library:371" deviceset="+5V" device=""/>
 <part name="LIPO" library="Connector" library_urn="urn:adsk.eagle:library:16378166" deviceset="2828XX-2" device="282834-2" package3d_urn="urn:adsk.eagle:package:24957623/2"/>
 <part name="GND1" library="supply1" library_urn="urn:adsk.eagle:library:371" deviceset="GND" device=""/>
-<part name="P+5" library="supply1" library_urn="urn:adsk.eagle:library:371" deviceset="+5V" device=""/>
 <part name="C1" library="SparkFun-Capacitors" library_urn="urn:adsk.eagle:library:510" deviceset="10NF" device="-0603-50V-10%" package3d_urn="urn:adsk.eagle:package:41385090/1" value="10nF"/>
 <part name="5V" library="Connector" library_urn="urn:adsk.eagle:library:16378166" deviceset="2828XX-2" device="282834-2" package3d_urn="urn:adsk.eagle:package:24957623/2"/>
@@
 <part name="GPIO" library="Connector" library_urn="urn:adsk.eagle:library:16378166" deviceset="PINHD-1X4" device="" package3d_urn="urn:adsk.eagle:package:22407/2"/>
 <part name="BATT" library="TL2285EE" deviceset="TL2285EE" device="" override_package3d_urn="urn:adsk.eagle:package:43003845/2" override_package_urn="urn:adsk.eagle:footprint:43003846/1"/>
-<part name="J2" library="53261-0871" deviceset="53261-0871" device=""/>
+<part name="J2" library="53261-0871" deviceset="53261-0871" device="" override_package3d_urn="urn:adsk.eagle:package:44544855/2" override_package_urn="urn:adsk.eagle:footprint:44544856/1"/>
 <part name="GND19" library="supply1" library_urn="urn:adsk.eagle:library:371" deviceset="GND" device=""/>
 </parts>
@@
 <attribute name="VALUE" x="-127" y="379.73" size="1.778" layer="96" rot="R90"/>
 </instance>
-<instance part="P+1" gate="1" x="-136.652" y="284.226" smashed="yes">
-<attribute name="VALUE" x="-139.192" y="279.146" size="1.778" layer="96" rot="R90"/>
-</instance>
 <instance part="LIPO" gate="G$1" x="-170.18" y="287.02" smashed="yes">
 <attribute name="VALUE" x="-170.18" y="284.226" size="1.778" layer="96" align="top-center"/>
@@
 <attribute name="VALUE" x="-180.34" y="273.558" size="1.778" layer="96"/>
 </instance>
-<instance part="P+5" gate="1" x="61.468" y="294.386" smashed="yes">
-<attribute name="VALUE" x="58.928" y="289.306" size="1.778" layer="96" rot="R90"/>
-</instance>
 <instance part="5V" gate="G$1" x="53.34" y="208.28" smashed="yes">

Commit message: JLCPCB V2
Parts:
- added C4: 100nf, 06035C104K4T2A:06035C104K4T2A
- added DW01: DW01-P, DW01-P:DW01-P
- added Q8: FS8205, FS8205:FS8205
- added R10: 100R, SparkFun-Resistors:1.20KOHM-0603-1/10W-1%
- added R9: 1k, SparkFun-Resistors:1.20KOHM-0603-1/10W-1%
- IP5306: value (none) -> IP5306
- R16, R4: value 470 -> 470R
- R6: value 15 -> 15k
- renumbered U$2 to IP5306
Connections:
- new net BATT-: C4.2, DW01.GND, LIPO.2, Q8.S1
- new net N$19: DW01.OC, Q8.G2
- new net N$37: C4.1, DW01.VCC, R10.1
- new net N$47: DW01.CS, R9.1
- new net N$9: DW01.OD, Q8.G1
- net GND: now also Q8.S2, R9.2; no longer LIPO.2
- net LBV: now also R10.2
Other:
- moved on the sheet: BATT, LIPO, PO, R14, R3, R8
