File: src/AQ_sensor_GSM.sch (EAGLE design)
At the start: 313 parts, among them J1 F-1X03-SIP-100-32, J2 53261-0871, J3 DS1021-1X2SF162-B, J4 S8411-45R, Q2 MMBT2222, Q3 MMBT2222, Q4 MMBT2222, Q5 MMBT2222, Q6 MMBT2222, Q7 MMBT2222, Q8 FS8205, T1 S8050, T2 S8050, U1 CP2102N-A02-GQFN28, U2 DS1307Z, U3 TP4056, U4 TPS63802DLAR, U5 TXS0108EPWR, U6 TPS63802DLAR, U7 TPS63802DLAR, U8 AMS1117-3.3, U9 AMS1117-1.8, X1 ESP32-S3-WROOM-1-N16R8, Y1 32.768kHz

Commit message: Update Sheet frames
Other:
- note added: "Designed by: Augustine Mwendwa Git: https://github.com/augustinemwendwa72 Email: augustinemwendwa72@gmail.com"
- note added: "LAST UPDATE: 30/April/2026"
- note added: "Name: Leds/ Buttons"
- note added: "Sheet Name: Clock"
- note added: "Sheet Name: Controller"
- note added: "Sheet Name: EC200UCN"
- note added: "Sheet Name: Logic Level"
- note added: "Sheet Name: Lora"
- note added: "Sheet Name: POWER"
- note added: "Sheet Name: Protection"
- note added: "sensors.AFRICA AQ Sensor"
- note removed: "LAST UPDATE: 21/5/2020"
- note removed: "LED AND BUTTONS"
- note removed: "sensors.AFRICA MRC"
- moved on the sheet: 12V, 12V_LED, 3.7_JST, 5V_IN, 5V_JST, 5V_LED, 5V_REG_1, AE1, BT_ANT, C10, C11, C12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
