File: src/AQ_sensor_GSM.s#h.sch (EAGLE design)
At the start: 161 parts, among them J1 F-1X03-SIP-100-32, J2 53261-0871, J3 PJ-002BH, J4 S8411-45R, Q2 MMBT2222, Q3 MMBT2222, Q4 MMBT2222, Q5 MMBT2222, Q6 MMBT2222, Q7 MMBT2222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

Commit message: Differential Pair routing
Parts:
- removed GSM_ANT1: (no value), SparkFun-Connectors:CONN_01
- removed J4: S8411-45R, S8411-45R:S8411-45R
- removed R41, R6: 0R, rcl:R-EU_R0603
- removed R44, R45, R50: 47K, rcl:R-EU_R0603
- removed U$1: SX1278, sx1278S2:SX1278
- removed U2: DS1307Z, SparkFun-Clocks:DS1307Z
- removed Y1: 32.768kHz, SparkFun-Clocks:CRYSTAL-32.768KHZSMD-3.2X1.5
Connections:
- net EUART_N renamed EUART_D-
- net EUART_P renamed EUART_D+
- net EUSB_N renamed EUSB_D-
- net EUSB_P renamed EUSB_D+
- net G_USB_N renamed G_USB_D-
- net G_USB_P renamed G_USB_D+
- removed net L_MIS0: U$1.MISO, X1.IO2
- removed net L_MOSI: U$1.MOSI, X1.IO1
- removed net L_NRESET: U$1.NRESET, X1.IO47
- removed net L_NSS: U$1.NSS, X1.IO46
- removed net L_SCK: U$1.SCK, X1.IO3
- removed net N$35: R6.2, U$1.ANT/NC
- removed net N$50: U2.X1, Y1.2
- removed net N$51: U2.X2, Y1.1
- removed net N$58: J4.+, U2.VBATT
- removed net N$59: J4.-, U2.GND
- removed net N$6: GSM_ANT1.1, R6.1
- removed net N$63: R41.1, U2.VCC
- removed net RTC_SCL: R45.2, U2.SCL, X1.IO13
- removed net RTC_SDA: R50.2, U2.SDA, X1.IO12
- removed net RTC_SQW: R44.2, U2.SQW, X1.IO48
- new net +5V: C33.2, C34.2, R46.1, U1.VREGIN
- new net IO1: X1.IO1
- new net IO12: X1.IO12
- new net IO13: X1.IO13
- new net IO2: X1.IO2
- new net IO3: X1.IO3
- new net IO46: X1.IO46
- new net IO47: X1.IO47
- new net IO48: X1.IO48
- net +3V3: no longer U$1.VDD3_3
- net 5V_OUT: no longer C33.2, C34.2, R41.2, R44.1, R45.1, R46.1, R50.1, U1.VREGIN
- net GND: no longer U$1.GND, U$1.GND1, U$1.GND2
Other:
- note removed: "Lora: https://www.lcsc.com/datasheet/lcsc_datasheet_2404121542_DreamLNK-M-SX1278S2_C845532.pdf"
