File: src/BCKP/AQ_sensor_GSM.brd (EAGLE design)
At the start: 110 x 64 mm, 113 parts, among them J1 F-1X03-SIP-100-32, J2 53261-0871, J3 PJ-002BH, Q2 MMBT2222, Q3 MMBT2222, Q4 MMBT2222, Q5 MMBT2222, Q6 MMBT2222, Q7 MMBT2222, U3 TEXAS_INSTRUMENTS_LM1117IMP-3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

Commit message: Routed
Parts:
- removed C23: TAJB106K016RNJ, Resistor_Capacitor:CAP_TANT_B
- removed R17: 2R, SparkFun-Resistors:0603
Connections:
- removed net N$13: C23.1, R17.1
- net 5V_IN: no longer R17.2
- net GND: no longer C23.2
- net USIM_VDD: no longer SIMCARD.C1
Changed lines of the file:
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@@
 <param name="PrefDir.14" value="0"/>
 <param name="PrefDir.15" value="0"/>
-<param name="PrefDir.16" value="|"/>
+<param name="PrefDir.16" value="*"/>
 <param name="cfVia" value="8"/>
 <param name="cfNonPref" value="5"/>
@@
 <attribute name="PROD_ID" value="RES-08413" x="40.862" y="20.6708" size="1.778" layer="28" rot="MR90" display="off"/>
 <attribute name="VALUE" x="40.1" y="20.6708" size="0.6096" layer="28" font="vector" ratio="20" rot="MR90" align="top-center"/>
-</element>
-<element name="C23" library="Resistor_Capacitor" library_urn="urn:adsk.eagle:library:15122775" package="CAP_TANT_B" package3d_urn="urn:adsk.eagle:package:10872905/4" value="TAJB106K016RNJ" x="72.0596" y="46.864" smashed="yes" rot="MR90" grouprefs="CHARGE_BOOST">
-<attribute name="CREATED_BY" value="PCBLayout.com" x="72.0596" y="46.864" size="1.778" layer="28" rot="MR90" display="off"/>
-<attribute name="DIGIKEY_PART_NUMBER" value="478-1673-2-ND" x="72.0596" y="46.864" size="1.778" layer="28" rot="MR90" display="off"/>
-<attribute name="MANUFACTURER" value="AVX Corporation" x="72.0596" y="46.864" size="1.778" layer="28" rot="MR90" display="off"/>
-<attribute name="MPN" value="TAJB106K016RNJ" x="72.0596" y="46.864" size="1.778" layer="28" rot="MR90" display="off"/>
-<attribute name="NAME" x="74.4916" y="45.532" size="1.2" layer="26" ratio="10" rot="MR90"/>
-<attribute name="PACKAGE" value="CAP TANT B" x="72.0596" y="46.864" size="1.778" layer="28" rot="MR90" display="off"/>
-<attribute name="VALUE" x="69.0116" y="44.832" size="1.2" layer="28" ratio="10" rot="MR90"/>
-</element>
-<element name="R17" library="SparkFun-Resistors" library_urn="urn:adsk.eagle:library:532" package="0603" package3d_urn="urn:adsk.eagle:package:39650/1" value="2R" x="79.4654" y="42.7688" smashed="yes" rot="MR90" grouprefs="CHARGE_BOOST">
-<attribute name="NAME" x="77.5096" y="42.972" size="0.6096" layer="26" font="vector" ratio="20" rot="MR90" align="bottom-center"/>
-<attribute name="PROD_ID" value="RES-08413" x="79.4654" y="42.7688" size="1.778" layer="28" rot="MR90" display="off"/>
-<attribute name="VALUE" x="78.7034" y="42.7688" size="0.6096" layer="28" font="vector" ratio="20" rot="MR90" align="top-center"/>
 </element>
 <element name="25%" library="led" library_urn="urn:adsk.eagle:library:259" package="CHIP-LED0603" package3d_urn="urn:adsk.eagle:package:15819/3" value="ORANGE" x="3.0988" y="25.7048" smashed="yes" rot="R90" grouprefs="CHARGING_LED WHOLE_PCB">
@@
 <contactref element="MT2492" pad="2"/>
 <contactref element="R6" pad="1"/>
-<contactref element="C23" pad="2"/>
 <contactref element="C30" pad="2"/>
 <contactref element="U$2" pad="9"/>
@@
 <wire x1="79.4368" y1="49.1112" x2="84.1682" y2="49.2738" width="0" layer="19" extent="1-16"/>
 <wire x1="77.343" y1="48.2724" x2="79.4368" y2="49.1112" width="0" layer="19" extent="1-16"/>
-<wire x1="72.0596" y1="48.339" x2="77.343" y2="48.2724" width="0" layer="19" extent="1-16"/>
-<wire x1="67.564" y1="48.3232" x2="72.0596" y2="48.339" width="0" layer="19" extent="1-16"/>
-<wire x1="64.916" y1="49.7188" x2="67.564" y2="48.3232" width="0" layer="19" extent="1-16"/>
-<wire x1="57.5822" y1="48.3776" x2="64.916" y2="49.7188" width="0" layer="19" extent="1-16"/>
 <wire x1="104.8468" y1="16.735" x2="97.6414" y2="19.0682" width="0" layer="19" extent="1-1"/>
 <wire x1="105.984" y1="15.088" x2="104.8468" y2="16.735" width="0" layer="19" extent="1-16"/>
@@
 <wire x1="106.1774" y1="35.2844" x2="98.7784" y2="36.9962" width="0" layer="19" extent="1-16"/>
 <wire x1="109.1274" y1="35.2844" x2="106.1774" y2="35.2844" width="0" layer="19" extent="1-1"/>
+<wire x1="67.564" y1="48.3232" x2="77.343" y2="48.2724" width="0" layer="19" extent="1-1"/>
+<wire x1="64.916" y1="49.7188" x2="67.564" y2="48.3232" width="0" layer="19" extent="1-16"/>
+<wire x1="57.5822" y1="48.3776" x2="64.916" y2="49.7188" width="0" layer="19" extent="1-16"/>
 <wire x1="54.1136" y1="40.6176" x2="57.5822" y2="48.3776" width="0" layer="19" extent="1-1"/>
 <wire x1="57.2228" y1="36.3766" x2="54.1136" y2="40.6176" width="0" layer="19" extent="1-1"/>
@@
 <wire x1="40.2238" y1="50.6872" x2="33.9106" y2="50.6108" width="0" layer="19" extent="16-16"/>
 </signal>
-<signal name="+3V3" class="1">
+<signal name="+3V3" class="3">
 <contactref element="SV1" pad="1"/>
 <contactref element="J1" pad="3"/>
@@
 <contactref element="D3" pad="1"/>
 <contactref element="EC200_GSM" pad="14"/>
-<contactref element="SIMCARD" pad="C1"/>
-<wire x1="64.7922" y1="17.6588" x2="84.1682" y2="48.0038" width="0" layer="19" extent="1-16"/>
 <wire x1="66.1414" y1="12.5682" x2="64.7922" y2="17.6588" width="0" layer="19" extent="1-16"/>
 <wire x1="58.4814" y1="12.328" x2="66.1414" y2="12.5682" width="0" layer="19" extent="1-1"/>
@@
 <wire x1="69.0198" y1="9.2238" x2="68.6168" y2="13.6958" width="0" layer="19" extent="16-16"/>
 <wire x1="48.0585" y1="19.624" x2="68.6168" y2="13.6958" width="0" layer="19" extent="16-16"/>
-</signal>
-<signal name="N$13">
-<contactref element="R17" pad="1"/>
-<contactref element="C23" pad="1"/>
-<wire x1="72.0596" y1="45.389" x2="79.4654" y2="41.9188" width="0" layer="19" extent="16-16"/>
 </signal>
 <signal name="N$14">
@@
 <contactref element="C21" pad="1"/>
 <contactref element="U$2" pad="1"/>
-<contactref element="R17" pad="2"/>
 <contactref element="C30" pad="1"/>
 <contactref element="5V" pad="1"/>
-<wire x1="87.4893" y1="17.8054" x2="79.4654" y2="43.6188" width="0" layer="19" extent="16-16"/>
-<wire x1="95.4752" y1="18.0412" x2="87.4893" y2="17.8054" width="0" layer="19" extent="16-16"/>
+<wire x1="87.4893" y1="17.8054" x2="95.4752" y2="18.0412" width="0" layer="19" extent="16-16"/>
 <wire x1="70.3168" y1="13.6958" x2="87.4893" y2="17.8054" width="0" layer="19" extent="16-16"/>
 <wire x1="70.0198" y1="9.2238" x2="70.3168" y2="13.6958" width="0" layer="19" extent="16-16"/>

Commit message: JLCPCB V2
Parts:
- added C23: TAJB106K016RNJ, Resistor_Capacitor:CAP_TANT_B
- added C4: 100nf, 06035C104K4T2A:CAPC1608X90N
- added Q1: FS8205A, FS8205A:SOP65P640X120-8N
- added R10: 100R, SparkFun-Resistors:0603
- added R17: 2R, SparkFun-Resistors:0603
- added R9: 1k, SparkFun-Resistors:0603
- added U1: DW01-P, DW01-P:SOT23-6L
- SV1, SV2: value (none) -> ZX-PM2.54-1-15PY
- moved Q3 100.6 mm to (3.79, 11.0), flipped to the top, turned to 90 degrees
- moved R22 100.0 mm to (9.08, 8.44), flipped to the top, turned to 90 degrees
- moved Q2 98.0 mm to (17.0, 8.75), flipped to the top
- moved R18 84.6 mm to (28.6, 8.69), flipped to the top, turned to 90 degrees
- moved R37 82.7 mm to (10.3, 21.8)
- moved U$2 67.8 mm to (17.8, 26.4)
- moved R20 66.0 mm to (15.5, 17.5), turned to 0 degrees
- moved R29 65.0 mm to (70.4, 17.6)
- moved C17 62.6 mm to (61.8, 8.58), flipped to the top, turned to 180 degrees
- moved C16 59.0 mm to (103.9, 43.6), flipped to the bottom, turned to 90 degrees
- moved C30 58.0 mm to (38.3, 25.9)
- moved C1 51.4 mm to (60.9, 3.12), flipped to the top, turned to 0 degrees
- moved R19 42.2 mm to (32.8, 18.3), turned to 90 degrees
- moved C24 40.7 mm to (24.6, 18.9), turned to 90 degrees
- moved R31 39.8 mm to (45.3, 8.30), flipped to the top, turned to 270 degrees
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Connections:
- new net BATT-: C4.2, LIPO.2, Q1.2, Q1.3, U1.6
- new net N$13: C23.1, R17.1
- new net N$19: Q1.5, U1.3
- new net N$37: C4.1, R10.1, U1.5
- new net N$47: R9.1, U1.2
- new net N$9: Q1.4, U1.1
- net 5V_IN: now also R17.2
- net GND: now also C23.2, Q1.6, Q1.7, R9.2; no longer LIPO.2
- net LBV: now also R10.2
- net USIM_VDD: now also SIMCARD.C1
Routing:
- net GND: track 0.00 -> 936.4 mm, vias 0 -> 20
- net V_LIPO: track 0.00 -> 231.7 mm, vias 0 -> 13
- net N$44: track 0.00 -> 214.9 mm, vias 0 -> 7
- net +3V3: track 0.00 -> 185.8 mm, vias 0 -> 8
- net G_ADC0: track 0.00 -> 162.2 mm, vias 0 -> 1
- net G_I2C_SDA: track 0.00 -> 158.6 mm, vias 0 -> 4
- net MCU_RXD: track 0.00 -> 151.0 mm, vias 0 -> 2
- net SIMCLK: track 0.00 -> 141.2 mm, vias 0 -> 11
- net G_ADC1: track 0.00 -> 138.3 mm, vias 0 -> 5
- net G_I2C_SCL: track 0.00 -> 138.0 mm, vias 0 -> 5
- net GSM_RST: track 0.00 -> 135.4 mm, vias 0 -> 3
- net 5V_OUT: track 0.00 -> 127.6 mm, vias 0 -> 6
- net G_USB_BOOT: track 0.00 -> 125.6 mm, vias 0 -> 5
- net MCU_DTR: track 0.00 -> 125.2 mm, vias 0 -> 5
- net 5V_IN: track 0.00 -> 123.8 mm, vias 0 -> 7
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Other:
- board size 110 x 64 mm -> 110.2 x 66.3 mm
