File: src/BCKP/AQ_sensor_GSM.sch (EAGLE design)
At the start: 111 parts, among them J1 F-1X03-SIP-100-32, J2 53261-0871, J3 PJ-002BH, Q2 MMBT2222, Q3 MMBT2222, Q4 MMBT2222, Q5 MMBT2222, Q6 MMBT2222, Q7 MMBT2222, U3 TEXAS_INSTRUMENTS_LM1117IMP-3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

Commit message: JLCPCB V2
Parts:
- added C23: TAJB106K016RNJ, Resistor_Capacitor:TAJB106K016RNJ
- added C4: 100nf, 06035C104K4T2A:06035C104K4T2A
- added Q1: FS8205A, FS8205A:FS8205A
- added R10: 100R, SparkFun-Resistors:1.20KOHM-0603-1/10W-1%
- added R17: 2R, SparkFun-Resistors:1.20KOHM-0603-1/10W-1%
- added R9: 1k, SparkFun-Resistors:1.20KOHM-0603-1/10W-1%
- added U1: DW01-P, DW01-P:DW01-P
- SV1, SV2: value (none) -> ZX-PM2.54-1-15PY
Connections:
- new net BATT-: C4.2, LIPO.2, Q1.S1, U1.GND
- new net N$13: C23.1, R17.1
- new net N$19: Q1.G2, U1.OC
- new net N$37: C4.1, R10.1, U1.VCC
- new net N$47: R9.1, U1.CS
- new net N$9: Q1.G1, U1.OD
- net 5V_IN: now also R17.2
- net GND: now also C23.2, Q1.S2, R9.2; no longer LIPO.2
- net LBV: now also R10.2
Other:
- moved on the sheet: PO, R14
