File: ESPS3_QuectelEC200U/V5/src/AQ_sensor_GSM.brd (EAGLE design)
At the start: 110.2 x 66.3 mm, 160 parts, among them J1 F-1X03-SIP-100-32, J2 53261-0871, J3 PJ-002BH, J4 S8411-45R, Q2 MMBT2222, Q3 MMBT2222, Q4 MMBT2222, Q5 MMBT2222, Q6 MMBT2222, Q7 MMBT2222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

Commit message: V5 revised
Parts:
- removed BATT: 2828XX-2282834-2, Connector:TERMBLK_254-2N
- added J5: B2B-XH-A, B2B-XH-A:JST_B2B-XH-A
- added RST2: SKRTLAE010, SKRTLAE010:SW_SKRTLAE010
- GSM_ANT: value (none) -> 1.9Ghz - 2.4Ghz
- moved R16 10.4 mm to (21.3, 11.8), turned to 90 degrees
- moved DHT 10.4 mm to (23.5, 11.7), turned to 0 degrees
- moved R24 6.70 mm to (33.5, 8.43), turned to 270 degrees
- moved Q4 5.83 mm to (37.7, 8.64), turned to 0 degrees
- moved R5 3.77 mm to (18.8, 11.8)
- moved 5V 0.99 mm to (22.6, 60.0)
Connections:
- net G_ADC2 renamed N$135
- net G_SPI_CLK renamed N$137
- net G_SPI_CS renamed N$136
- net G_SPI_MISO renamed N$134
- net G_SPI_MOSI renamed N$83
- net SDIO1_VDD renamed N$90
- net VPP renamed N$113
- removed net SHIELD: MICRO_SD1.MP1, MICRO_SD1.MP2, MICRO_SD1.MP3, MICRO_SD1.MP4
- new net N$100: EC200_GSM.79
- new net N$101: EC200_GSM.80
- new net N$102: EC200_GSM.75
- new net N$103: EC200_GSM.77
- new net N$104: EC200_GSM.142
- new net N$105: EC200_GSM.141
- new net N$106: EC200_GSM.4
- new net N$107: EC200_GSM.1
- new net N$108: EC200_GSM.23
- new net N$109: EC200_GSM.140
- new net N$112: EC200_GSM.3
- new net N$114: U1.17
- new net N$115: U1.16
- new net N$116: U1.22
- new net N$117: U1.21
- new net N$118: U1.20
- new net N$119: U1.27
- new net N$120: U1.23
- new net N$121: U1.14
- new net N$122: U1.15
- new net N$123: U1.13
- new net N$124: U1.12
- new net N$125: U1.11
- new net N$126: U1.2
- new net N$127: U1.1
- new net N$128: U$1.5
- new net N$129: U$1.6
- new net N$130: U$1.7
- new net N$131: U$1.8
- new net N$132: U$1.10
- new net N$133: U$1.11
- new net N$15: EC200_GSM.113
- new net N$16: EC200_GSM.114
- new net N$23: EC200_GSM.73
- new net N$5: EC200_GSM.83
- new net N$60: EC200_GSM.74
- new net N$64: EC200_GSM.121
- new net N$65: EC200_GSM.119
- new net N$66: EC200_GSM.123
- new net N$67: EC200_GSM.122
- new net N$68: EC200_GSM.120
- new net N$69: EC200_GSM.124
- new net N$70: EC200_GSM.125
- new net N$73: EC200_GSM.118
- new net N$75: EC200_GSM.143
- new net N$76: EC200_GSM.144
- new net N$77: EC200_GSM.132
- new net N$78: EC200_GSM.131
- new net N$79: EC200_GSM.130
- new net N$8: EC200_GSM.84
- new net N$80: EC200_GSM.129
- new net N$81: EC200_GSM.134
- new net N$82: EC200_GSM.133
- new net N$84: EC200_GSM.32
- new net N$85: EC200_GSM.33
- new net N$86: EC200_GSM.28
- new net N$87: EC200_GSM.29
- new net N$88: EC200_GSM.30
- new net N$89: EC200_GSM.31
- new net N$91: EC200_GSM.25
- new net N$92: EC200_GSM.26
- new net N$93: EC200_GSM.24
- new net N$94: EC200_GSM.27
- new net N$95: EC200_GSM.137
- new net N$96: EC200_GSM.138
- new net N$97: EC200_GSM.11
- new net N$98: EC200_GSM.12
- new net N$99: EC200_GSM.78
- net BATT-: now also J5.1; no longer BATT.2
- net ESP_RST: now also RST2.1, RST2.3
- net GND: now also MICRO_SD1.MP1, MICRO_SD1.MP2, MICRO_SD1.MP3, MICRO_SD1.MP4, RST2.2, RST2.S1, RST2.S2
- net LBV: now also J5.2; no longer BATT.1
Routing:
- net ESP_RST: track 102.9 -> 157.4 mm, vias 5 -> 8
- net SHIELD: track 42.4 -> 0.00 mm, vias 4 -> 0
- net N$26: track 40.3 -> 48.5 mm
- net +3V3: track 238.7 -> 245.5 mm
- net N$14: track 62.4 -> 55.8 mm
- net N$29: track 55.3 -> 61.1 mm
- net GND: track 409.1 -> 413.5 mm, vias 130 -> 128
- net DHT_LED: track 88.7 -> 92.7 mm
- net BATT-: track 51.3 -> 48.6 mm
- net GSM_RST_O: track 68.9 -> 71.5 mm
- net GSM_RST: track 61.8 -> 64.1 mm
- net N$18: track 58.2 -> 56.3 mm
- net L_NSS: track 111.4 -> 112.7 mm
- net 5V_IN: track 112.1 -> 113.2 mm
- net DHT_OUT: track 95.2 -> 96.0 mm
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Other:
- board text added: "3.7v"
