File: ESPS3_QuectelEC200U/V5/src/AQ_sensor_GSM.sch (EAGLE design)
At the start: 161 parts, among them J1 F-1X03-SIP-100-32, J2 53261-0871, J3 PJ-002BH, J4 S8411-45R, J5 B2B-XH-A, Q2 MMBT2222, Q3 MMBT2222, Q4 MMBT2222, Q5 MMBT2222, Q6 MMBT2222, Q7 MMBT2222, Q8 FS8205, T1 S8050, T2 S8050, U1 CP2102N-A02-GQFN28, U2 DS1307Z, U5 TXS0108EPWR, X1 ESP32-S3-WROOM-1-N16R8, Y1 32.768kHz

Commit message: V5 revised
Parts:
- added U$10, U$11, U$12, U$13, U$14, U$15, U$16, U$17, U$18, U$19, U$2, U$20, U$21, U$22, U$23, U$24, U$25, U$26, U$27, U$28, U$29, U$3, U$30, U$31, U$32, U$33, U$34, U$35, U$36, U$37, U$38, U$39, U$4, U$40, U$41, U$42, U$43, U$44, U$45, U$46, U$47, U$48, U$49, U$5, U$50, U$51, U$52, U$53, U$54, U$55, U$56, U$57, U$58, U$59, U$6, U$60, U$61, U$62, U$63, U$64, U$65, U$66, U$67, U$68, U$69, U$7, U$70, U$71, U$72, U$73, U$74, U$75, U$76, U$77, U$78, U$79, U$8, U$80, U$81, U$82, U$83, U$84, U$9: NC_MARKER, NC_MARKER:NC_MARKER
Connections:
- removed net G_ADC2: EC200_GSM.ADC2
- removed net G_SPI_CLK: EC200_GSM.SPI_CLK
- removed net G_SPI_CS: EC200_GSM.SPI_CS
- removed net G_SPI_MISO: EC200_GSM.SPI_MISO
- removed net G_SPI_MOSI: EC200_GSM.SPI_MOSI
- new net N$100: EC200_GSM.KEYIN2, U$44.P$1
- new net N$101: EC200_GSM.KEYIN3, U$43.P$1
- new net N$102: EC200_GSM.MIC_P, U$42.P$1
- new net N$103: EC200_GSM.MIC_N, U$41.P$1
- new net N$104: EC200_GSM.I2C2_SDA, U$40.P$1
- new net N$105: EC200_GSM.I2C2_SCL, U$39.P$1
- new net N$106: EC200_GSM.!W_DISABLE, U$50.P$1
- new net N$107: EC200_GSM.WAKEUP_IN, U$51.P$1
- new net N$108: EC200_GSM.SD_DET, U$52.P$1
- new net N$109: EC200_GSM.ISINK, U$53.P$1
- new net N$110: EC200_GSM.AP_READY, U$54.P$1
- new net N$111: EC200_GSM.USIM2_VDD, U$57.P$1
- new net N$112: EC200_GSM.SLEEP_IND, U$56.P$1
- new net N$113: SIMCARD.VPP, U$58.P$1
- new net N$114: U$70.P$1, U1.GPIO.2/RS485
- new net N$115: U$69.P$1, U1.GPIO.3/WAKEUP
- new net N$116: U$68.P$1, U1.GPIO.4
- new net N$117: U$67.P$1, U1.GPIO.5
- new net N$118: U$66.P$1, U1.GPIO.6
- new net N$119: U$65.P$1, U1.DSR
- new net N$120: U$64.P$1, U1.CTS
- new net N$121: U$63.P$1, U1.CHR1
- new net N$122: U$62.P$1, U1.CHR0
- new net N$123: U$61.P$1, U1.CHREN
- new net N$124: U$60.P$1, U1.SUSPEND
- new net N$125: U$59.P$1, U1.!SUSPEND
- new net N$126: U$73.P$1, U1.RI/CLK
- new net N$127: U$74.P$1, U1.DCD
- new net N$128: U$1.DIO0, U$75.P$1
- new net N$129: U$1.DIO1, U$76.P$1
- new net N$130: U$1.DIO2, U$77.P$1
- new net N$131: U$1.DIO3, U$78.P$1
- new net N$132: U$1.DIO4, U$80.P$1
- new net N$133: U$1.DIO5, U$79.P$1
- new net N$134: EC200_GSM.SPI_MISO, U$81.P$1
- new net N$135: EC200_GSM.ADC2, U$82.P$1
- new net N$136: EC200_GSM.SPI_CS, U$84.P$1
- new net N$137: EC200_GSM.SPI_CLK, U$83.P$1
- new net N$15: EC200_GSM.KEYOUT2, U$4.P$1
- new net N$16: EC200_GSM.KEYOUT3, U$5.P$1
- new net N$23: EC200_GSM.LOUDSPK_P, U$6.P$1
- new net N$5: EC200_GSM.KEYOUT0, U$2.P$1
- new net N$60: EC200_GSM.LOUDSPK_N, U$7.P$1
- new net N$64: EC200_GSM.LCD_SEL, U$8.P$1
- new net N$65: EC200_GSM.LCD_FMARK, U$9.P$1
- new net N$66: EC200_GSM.LCD_CLK, U$10.P$1
- new net N$67: EC200_GSM.LCD_CS, U$11.P$1
- new net N$68: EC200_GSM.LCD_RSTB, U$12.P$1
- new net N$69: EC200_GSM.LCD_SDC, U$13.P$1
- new net N$7: EC200_GSM.BT_EN, U$55.P$1
- new net N$70: EC200_GSM.LCD_SI/O, U$14.P$1
- new net N$71: EC200_GSM.WLAN_EN, U$15.P$1
- new net N$72: EC200_GSM.WLAN_PWR_EN, U$16.P$1
- new net N$73: EC200_GSM.WLAN_SLP_CLK, U$17.P$1
- new net N$74: EC200_GSM.WLAN_WAKE, U$18.P$1
- new net N$75: EC200_GSM.GRFC1, U$19.P$1
- new net N$76: EC200_GSM.GRFC2, U$20.P$1
- new net N$77: EC200_GSM.SDIO2_DATA0, U$21.P$1
- new net N$78: EC200_GSM.SDIO2_DATA1, U$23.P$1
- new net N$79: EC200_GSM.SDIO2_DATA2, U$22.P$1
- new net N$8: EC200_GSM.KEYOUT1, U$3.P$1
- new net N$80: EC200_GSM.SDIO2_DATA3, U$24.P$1
- new net N$81: EC200_GSM.SDIO2_CMD, U$25.P$1
- new net N$82: EC200_GSM.SDIO2_CLK, U$26.P$1
- new net N$83: EC200_GSM.SPI_MOSI, U$27.P$1
- new net N$84: EC200_GSM.SDIO1_CLK, U$28.P$1
- new net N$85: EC200_GSM.SDIO1_CMD, U$29.P$1
- new net N$86: EC200_GSM.SDIO1_DATA3, U$30.P$1
- new net N$87: EC200_GSM.SDIO1_DATA2, U$31.P$1
- new net N$88: EC200_GSM.SDIO1_DATA1, U$32.P$1
- new net N$89: EC200_GSM.SDIO1_DATA0, U$33.P$1
- new net N$90: EC200_GSM.SDIO1_VDD, U$34.P$1
- new net N$91: EC200_GSM.PCM_DOUT, U$35.P$1
- new net N$92: EC200_GSM.PCM_SYNC, U$36.P$1
- new net N$93: EC200_GSM.PCM_DIN, U$37.P$1
- new net N$94: EC200_GSM.PCM_CLK, U$38.P$1
- new net N$95: EC200_GSM.AUX_RXD, U$49.P$1
- new net N$96: EC200_GSM.AUX_TXD, U$48.P$1
- new net N$97: EC200_GSM.DBG_RXD, U$47.P$1
- new net N$98: EC200_GSM.DBG_TXD, U$46.P$1
- new net N$99: EC200_GSM.KEYIN1, U$45.P$1
- net GND: now also MICRO_SD1.SHIELD
