File: ESPS3_QuectelEC200U/V4/src/AQ_sensor_GSM.brd (EAGLE design)
At the start: 110.2 x 66.3 mm, 160 parts, among them J1 F-1X03-SIP-100-32, J2 53261-0871, J3 PJ-002BH, J4 S8411-45R, Q2 MMBT2222, Q3 MMBT2222, Q4 MMBT2222, Q5 MMBT2222, Q6 MMBT2222, Q7 MMBT2222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

Commit message: V4 revised with images
Connections:
- net PMS_RX: now also X1.23; no longer X1.26
- net PMS_TX: now also X1.26; no longer X1.23
- net SD_MISO: now also X1.34; no longer X1.33
- net SD_MOSI: now also X1.33; no longer X1.34
Routing:
- net PMS_RX: track 15.9 -> 19.6 mm
- net PMS_TX: track 20.4 -> 17.0 mm
- net SD_MOSI: track 49.1 -> 50.3 mm
- net SD_MISO: track 40.1 -> 41.0 mm
- net MCU_DTR: track 9.03 -> 9.88 mm
- net MCU_RXD: track 21.1 -> 21.9 mm
