File: ESPS3_QuectelEC200U/V3/src/AQ_sensor_GSM.sch (EAGLE design)
At the start: 120 parts, among them IC1 MIC29302WU, J1 F-1X03-SIP-100-32, J3 PJ-002BH, Q1 MMBT2222, Q2 MMBT2222, Q3 MMBT2222, Q4 MMBT2222, Q5 MMBT2222, Q6 MMBT2222, Q7 MMBT2222, U3 TEXAS_INSTRUMENTS_LM1117IMP-3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, U5 TXS0108EPWR, X1 53048-08

Commit message: V3 revised
Parts:
- removed C12: 470uf, T495X477K010ATE100:T495X477K010ATE100
- removed C14: 22nF, SparkFun-Capacitors:220PF-0402T-50V-5%
- removed C22, C25, C26, C27: ECA-1HM220, Resistor_Capacitor:ECA-1HM220
- removed C7: 100nf, 06035C104K4T2A:06035C104K4T2A
- removed CHARGE: PCM12SMTR, AQ_sensor_MRC:PCM12SMTR
- removed D5: ESD56151W04, 4.7V TVS Diode:1N4148WS_RR
- removed IC1: MIC29302WU, MIC29302WU:MIC29302WU
- removed LIPO/BUCK, USB/BATT: TL2285EE, TL2285EE:TL2285EE
- removed POWER: RED, led:LEDCHIP-LED0603
- removed Q1: MMBT2222, MMBT2222_:MMBT2222
- removed R1: 110k, SparkFun-Resistors:1.20KOHM-0603-1/10W-1%
- removed R11: 470R, rcl:R-EU_R0603
- removed R6: 15, SparkFun-Resistors:1.20KOHM-0603-1/10W-1%
- removed R7: 10k, SparkFun-Resistors:1.20KOHM-0603-1/10W-1%
- removed SOLAR_IN: 10118192-0001LF, AQ_sensor_GSM:10118192-0001LF
- removed U$1: (no value), MT2492:MT2492MT2492
- removed X1: 53048-08, AQ_sensor_GSM:53048-08
- added 5V: 2828XX-2282834-2, Connector:2828XX-2282834-2
- added 5V_PWR: RED, led:LEDCHIP-LED0603
- added BATT, PWR: TL2285EE, TL2285EE:TL2285EE
- added C4: 100nf, 06035C104K4T2A:06035C104K4T2A
- added CHARGER: KMR621NGLFS, AQ_sensor_GSM:KMR621NGLFS
- added D6: SS54-HF, SS54-HF schottkey Diode:SS54-HF
- added DW01: DW01-P, DW01-P:DW01-P
- added GPIO, PROG: PINHD-1X4, Connector:PINHD-1X4
- added J2: 53261-0871, 53261-0871:53261-0871
- added PWR_ON: ORANGE, led:LEDCHIP-LED0603
- added Q8: FS8205, FS8205:FS8205
- added R502: 10R, rcl:R-EU_R0603
- added VR1, VR2: LM7805MPX/NOPB, LM7805MPX_NOPB:LM7805MPX/NOPB
- C2: value 470uf -> 100uF; device T495X477K010ATE100:T495X477K010ATE100 -> rcl:CPOL-EUD
- C3: value 100nf -> 100pF; device 06035C104K4T2A:06035C104K4T2A -> SparkFun-Capacitors:100PF-0603-50V-5%
- C5: value ECA-1HM220 -> 100nf; device Resistor_Capacitor:ECA-1HM220 -> 06035C104K4T2A:06035C104K4T2A
- C6: value EEEFN1C471P -> 100uF; device EEEFN1C471P:EEEFN1C471P -> rcl:CPOL-EUD
- IP5306: value (none) -> IP5306
- L1: value 784787047 -> LQW15AN47NG00D; device Fixed Inductors:784787047 -> LQW15AN47NG00D 47uh:LQW15AN47NG00D
- R10: value 47K -> 100R; device rcl:R-EU_R0603 -> SparkFun-Resistors:1.20KOHM-0603-1/10W-1%
- R16, R4: value 470 -> 470R
- R2: value 51K -> 1k; device rcl:R-EU_R0603 -> SparkFun-Resistors:1.20KOHM-0603-1/10W-1%
- R3: value 4.7K -> 47k; device rcl:R-EU_R0603 -> SparkFun-Resistors:1.20KOHM-0603-1/10W-1%
- R8: value 47K -> 10k; device rcl:R-EU_R0603 -> SparkFun-Resistors:1.20KOHM-0603-1/10W-1%
- R9: value 100k -> 1k; device rcl:R-EU_R0603 -> SparkFun-Resistors:1.20KOHM-0603-1/10W-1%
- renumbered 10K to R501, 51K to R500, C_P to CHARGING, U$2 to IP5306
Connections:
- removed net +5V: R14.2, SV2.1, U3.IN, USB/BATT.COM1, USB/BATT.COM2, X1-8.S
- removed net 3.8V: C6.1, C7.2, D5.K, IC1.OUT, LIPO/BUCK.NC1, LIPO/BUCK.NC2, R11.2, R9.2
- removed net 4.2V: C29.1, IP5306.BAT, L2.2, LIPO/BUCK.NO1, LIPO/BUCK.NO2, R19.2
- removed net BVIN: C5.1, J3.1, R7.2, SOLAR_IN.VUSB, U$1.VIN
- removed net D+: PB_IN.D+, SOLAR_IN.D+
- removed net D-: PB_IN.D-, SOLAR_IN.D-
- removed net N$11: R7.1, U$1.EN
- removed net N$6: C14.2, L1.1, U$1.SW
- removed net TF-CLK: SV2.7
- removed net TF-CS: SV2.9
- removed net TF-MISO: SV2.8
- removed net TF-MOSI: SV2.10
- removed net VUSB: C2.1, C3.2, IC1.VIN, PB_IN.VUSB, R2.2, USB/BATT.NC1, USB/BATT.NC2
- new net 5VT: PB_IN.VUSB, PWR.NO1, PWR.NO2
- new net BATT-: C4.2, DW01.GND, LIPO.2, Q8.S1
- new net BMSV: R3.2, R8.1, SV2.15
- new net G_ADC0: EC200_GSM.ADC0, GPIO.1
- new net G_ADC1: EC200_GSM.ADC1, GPIO.2
- new net G_ADC2: EC200_GSM.ADC2
- new net G_GPIO1: EC200_GSM.GPIO1
- new net G_I2C_SCL: EC200_GSM.I2C_SCL, GPIO.4
- new net G_I2C_SDA: EC200_GSM.I2C_SDA, GPIO.3
- new net G_SPI_CLK: EC200_GSM.SPI_CLK
- new net G_SPI_CS: EC200_GSM.SPI_CS
- new net G_SPI_MISO: EC200_GSM.SPI_MISO
- new net G_SPI_MOSI: EC200_GSM.SPI_MOSI
- new net G_USB_BOOT: EC200_GSM.USB_BOOT, PROG.1
- new net G_USB_D+: EC200_GSM.USB_DP, PB_IN.D+
- new net G_USB_D-: EC200_GSM.USB_DM, PB_IN.D-
- new net G_USB_VBUS: EC200_GSM.USB_VBUS
- new net LBV: BATT.COM1, BATT.COM2, LIPO.1, R10.2, R3.1
- new net N$19: DW01.OC, Q8.G2
- new net N$47: DW01.CS, R9.1
- new net N$61: D6.A, J3.1
- new net N$9: DW01.OD, Q8.G1
- net 5V_IN: now also 5V.1, PWR.COM1, PWR.COM2, R2.1; no longer C22.1, L1.2, R1.2
- net 5V_OUT: now also C2.+, J2.8, R14.2, SV2.1, U3.IN; no longer C25.1, C26.1, C27.1, USB/BATT.NO1, USB/BATT.NO2
- net GND: now also 5V.2, 5V_PWR.C, C2.-, C21.2, C5.1, C6.-, CHARGER.2, J2.7, PROG.4, PWR_ON.C, Q8.S2, R8.2, R9.2, VR1.GND_2, VR1.GND_4, VR2.GND_2, VR2.GND_4; no longer C12.2, C2.2, C22.2, C25.2, C26.2, C27.2, C3.1, C5.2, C6.2, C7.1, CHARGE.2, D5.A, IC1.GND, LIPO.2, POWER.C, R10.1, R11.1, R6.1, R8.1, SOLAR_IN.GND, SOLAR_IN.ID, SOLAR_IN.SHIELD, U$1.GND, X1-7.S
- net GNSS_ANT: now also C3.2; no longer GPS.SIG
- net MCU_RXD: now also PROG.2
- net MCU_TXD: now also PROG.3
- net N$10: now also C3.1, GPS.SIG, L1.1; no longer C21.2, R1.1, R6.2, U$1.FB
- net N$20: now also CHARGER.1; no longer CHARGE.1
- net N$25: now also 5V_PWR.A; no longer POWER.A
- net N$3: now also L1.2, R502.1; no longer C14.1, U$1.BS
- net N$35: now also PWR_ON.A, R2.2; no longer IC1.EN, Q1.C, R2.1
- net N$36: now also D6.K, VR1.INPUT, VR2.INPUT; no longer Q1.B, R3.2
- net N$37: now also C4.1, DW01.VCC, R10.1; no longer Q1.E, R8.2
- net N$38: now also PWR.NC1, PWR.NC2, VR1.OUTPUT, VR2.OUTPUT; no longer IC1.ADJ, R10.2, R9.1
- net PMS_RX: now also J2.5; no longer X1-5.S
- net PMS_TX: now also J2.4; no longer X1-4.S
- net VBAT_EN: no longer R3.1
- net V_LIPO: now also BATT.NO1, BATT.NO2, C29.1, C5.2, C6.+, IP5306.BAT, L2.2, R19.2, R502.2; no longer C12.1, LIPO.1, LIPO/BUCK.COM1, LIPO/BUCK.COM2
Other:
- note added: "GSM RESET"
- note removed: "POWER KEY"
- moved on the sheet: C21, C8, GPS, J3, LIPO, R14, U3
