File: ESPS3_QuectelEC200U/V2/src/AQ_sensor_GSM.sch (EAGLE design)
At the start: 100 parts, among them IC1 MIC29302WU, IC2 MCP73831/OT, J1 F-1X03-SIP-100-32, J3 PJ-002BH, Q1 MMBT2222, Q2 MMBT2222, Q3 MMBT2222, Q4 MMBT2222, Q5 MMBT2222, Q6 MMBT2222, Q7 MMBT2222, U1 LM7805S/NOPB, U3 TEXAS_INSTRUMENTS_LM1117IMP-3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, U5 TXS0108EPWR, X1 53048-08

Commit message: V2 revised
Parts:
- removed 3.7V_LIPO: 2828XX-2282837-2, Connector:2828XX-2282837-2
- removed C6: EEEFN1C471P, EEEFN1C471P:EEEFN1C471P
- removed C7: 100nf, 06035C104K4T2A:06035C104K4T2A
- removed CHRG, POWER: RED, led:LEDCHIP-LED0603
- removed D5: ESD56151W04, 4.7V TVS Diode:1N4148WS_RR
- removed FULL: YELLOW, led:LEDCHIP-LED0603
- removed IC1: MIC29302WU, MIC29302WU:MIC29302WU
- removed IC2: MCP73831/OT, AQ_sensor_GSM:MCP73831/OT
- removed LIPO_SW, S1: TL2285EE, TL2285EE:TL2285EE
- removed MICRO_SD1: TF-01A, TF-01A:TF-01A
- removed MICRO_USB: 10118192-0001LF, AQ_sensor_GSM:10118192-0001LF
- removed Q1: MMBT2222, MMBT2222_:MMBT2222
- removed R11: 470R, rcl:R-EU_R0603
- removed U1: LM7805S/NOPB, LM7805S_NOPB:LM7805S/NOPB
- removed X1: 53048-08, AQ_sensor_GSM:53048-08
- added 100%, 25%, 50%, 75%, CHARGING, PWR_ON: ORANGE, led:LEDCHIP-LED0603
- added 5V, LIPO: 2828XX-2282834-2, Connector:2828XX-2282834-2
- added BATT, PWR: TL2285EE, TL2285EE:TL2285EE
- added C14: 22nF, SparkFun-Capacitors:220PF-0402T-50V-5%
- added C21: 22pF, SparkFun-Capacitors:220PF-0402T-50V-5%
- added C23, C24, C29, C30: TAJB106K016RNJ, Resistor_Capacitor:TAJB106K016RNJ
- added CHARGER: KMR621NGLFS, AQ_sensor_GSM:KMR621NGLFS
- added D4, D6, D7: SS54-HF, SS54-HF schottkey Diode:SS54-HF
- added DW01: DW01-P, DW01-P:DW01-P
- added GPIO, PROG: PINHD-1X4, Connector:PINHD-1X4
- added IP5306: IP5306, IP5306:IP5306IP5306
- added J2: 53261-0871, 53261-0871:53261-0871
- added L1: 784787047, Fixed Inductors:784787047
- added L2: 784778010, Fixed Inductors:784778010
- added MT2492: MT2492, MT2492:MT2492MT2492
- added PB_IN: 10118192-0001LF, AQ_sensor_GSM:10118192-0001LF
- added PO: RED, led:LEDCHIP-LED0603
- added Q8: FS8205, FS8205:FS8205
- added R1: 110k, SparkFun-Resistors:1.20KOHM-0603-1/10W-1%
- added R37, R7: 10k, SparkFun-Resistors:1.20KOHM-0603-1/10W-1%
- added R6: 15k, SparkFun-Resistors:1.20KOHM-0603-1/10W-1%
- C1: value 10uF -> 10nF; device rcl:C-EUC0603 -> SparkFun-Capacitors:10NF-0603-50V-10%
- C2: value 470uf -> 100uF; device T495X477K010ATE100:T495X477K010ATE100 -> rcl:CPOL-EUD
- C3: value 100nf -> 100uF; device 06035C104K4T2A:06035C104K4T2A -> rcl:CPOL-EUD
- C4: value 10uF -> 100nf; device rcl:C-EUC0603 -> 06035C104K4T2A:06035C104K4T2A
- R10: value 47K -> 100R; device rcl:R-EU_R0603 -> SparkFun-Resistors:1.20KOHM-0603-1/10W-1%
- R16, R4: value 470 -> 470R
- R17, R19: value 470 -> 2R; device rcl:R-EU_R0603 -> SparkFun-Resistors:1.20KOHM-0603-1/10W-1%
- R2: value 51K -> 1k; device rcl:R-EU_R0603 -> SparkFun-Resistors:1.20KOHM-0603-1/10W-1%
- R20: value 2K -> 220R; device rcl:R-EU_R0603 -> SparkFun-Resistors:1.20KOHM-0603-1/10W-1%
- R3: value 4.7K -> 47k; device rcl:R-EU_R0603 -> SparkFun-Resistors:1.20KOHM-0603-1/10W-1%
- R8: value 47K -> 10k; device rcl:R-EU_R0603 -> SparkFun-Resistors:1.20KOHM-0603-1/10W-1%
- R9: value 100k -> 1k; device rcl:R-EU_R0603 -> SparkFun-Resistors:1.20KOHM-0603-1/10W-1%
- renumbered GSMANTENNA2 to GSM_ANT, M_RI to MRI, N_MODE to NMDE, N_STAT to NST, P_STAT to PST
Connections:
- removed net +5V: C1.1, C2.1, C3.2, CHRG.A, IC1.VIN, IC2.VDD, R14.2, R2.2, S1.NO1, S1.NO2, SV2.1, U1.OUT, U3.IN, X1-8.S
- removed net BP: 3.7V_LIPO.2, IC2.VBAT, LIPO_SW.NC1, LIPO_SW.NC2
- removed net CP: C6.1, C7.2, D5.K, IC1.OUT, LIPO_SW.NO1, LIPO_SW.NO2, R11.2, R9.2
- removed net D+: MICRO_USB.D+
- removed net D-: MICRO_USB.D-
- removed net JACKP: J3.1, U1.IN
- removed net N$12: FULL.A, R19.1
- removed net N$36: Q1.B, R3.2
- removed net N$38: IC1.ADJ, R10.2, R9.1
- removed net TF-CLK: MICRO_SD1.CLK, SV2.7
- removed net TF-CS: MICRO_SD1.CD/DAT3, SV2.9
- removed net TF-MISO: MICRO_SD1.DAT0, SV2.8
- removed net TF-MOSI: MICRO_SD1.CMD, SV2.10
- removed net USBP: MICRO_USB.VUSB, S1.COM1, S1.COM2
- removed net VRTC: C4.1
- new net 4.5-16V: C3.+, MT2492.VIN, PWR.COM1, PWR.COM2, R2.1, R7.2
- new net 5VT: D4.K, PWR.NO1, PWR.NO2
- new net 5V_IN: 5V.1, C21.1, C30.1, IP5306.VIN, L1.2, R1.2, R17.2
- new net 5V_OUT: C2.+, IP5306.VOUT, J2.8, R14.2, SV2.1, U3.IN
- new net BATT-: C4.2, DW01.GND, LIPO.2, Q8.S1
- new net BMSV: R3.2, R8.1, SV2.15
- new net G_ADC0: EC200_GSM.ADC0, GPIO.1
- new net G_ADC1: EC200_GSM.ADC1, GPIO.2
- new net G_ADC2: EC200_GSM.ADC2
- new net G_GPIO1: EC200_GSM.GPIO1
- new net G_I2C_SCL: EC200_GSM.I2C_SCL, GPIO.4
- new net G_I2C_SDA: EC200_GSM.I2C_SDA, GPIO.3
- new net G_SPI_CLK: EC200_GSM.SPI_CLK
- new net G_SPI_CS: EC200_GSM.SPI_CS
- new net G_SPI_MISO: EC200_GSM.SPI_MISO
- new net G_SPI_MOSI: EC200_GSM.SPI_MOSI
- new net G_USB_BOOT: EC200_GSM.USB_BOOT, PROG.1
- new net G_USB_D+: EC200_GSM.USB_DP, PB_IN.D+
- new net G_USB_D-: EC200_GSM.USB_DM, PB_IN.D-
- new net G_USB_VBUS: EC200_GSM.USB_VBUS
- new net LBV: BATT.COM1, BATT.COM2, LIPO.1, R10.2, R3.1
- new net N$10: C21.2, MT2492.FB, R1.1, R6.2
- new net N$11: MT2492.EN, R7.1
- new net N$14: 100%.A, 25%.C, 50%.A, 75%.C, IP5306.LED3
- new net N$17: 25%.A, 50%.C, IP5306.LED1
- new net N$18: 100%.C, 75%.A, IP5306.LED2
- new net N$19: DW01.OC, Q8.G2
- new net N$20: CHARGER.1, R37.1
- new net N$21: IP5306.SW, L2.1
- new net N$24: C24.1, R19.1
- new net N$3: C14.1, MT2492.BS
- new net N$45: IP5306.KEY, R20.2, R37.2
- new net N$46: CHARGING.A, R20.1
- new net N$47: DW01.CS, R9.1
- new net N$59: D4.A, PB_IN.VUSB
- new net N$60: D7.K, J3.2, J3.3
- new net N$61: D6.A, J3.1
- new net VUSB: D6.K, PWR.NC1, PWR.NC2
- net +3V3: no longer MICRO_SD1.VDD
- net GND: now also 5V.2, C2.-, C23.2, C24.2, C29.2, C3.-, C30.2, CHARGER.2, CHARGING.C, D1.ANODE, D7.A, IP5306.GND, J2.7, MT2492.GND, PB_IN.GND, PB_IN.ID, PB_IN.SHIELD, PO.C, PROG.4, PWR_ON.C, Q8.S2, R6.1, R8.2, R9.2; no longer 3.7V_LIPO.1, C2.2, C3.1, C4.2, C6.2, C7.1, D1.CATHODE, D5.A, FULL.C, IC1.GND, IC2.VSS, J3.2, J3.3, MICRO_SD1.SHIELD, MICRO_SD1.VSS, MICRO_USB.GND, MICRO_USB.ID, MICRO_USB.SHIELD, POWER.C, R10.1, R11.1, R20.2, R8.1, U1.GND, X1-7.S
- net GSM_RST: now also D1.CATHODE, GSM_RST.2
- net MCU_RXD: now also PROG.2
- net MCU_TXD: now also PROG.3
- net N$13: now also C23.1, R17.1; no longer IC2.PROG, R20.1
- net N$25: now also PO.A; no longer POWER.A
- net N$35: now also PWR_ON.A, R2.2; no longer IC1.EN, Q1.C, R2.1
- net N$37: now also C4.1, DW01.VCC, R10.1; no longer Q1.E, R8.2
- net N$6: now also C14.2, L1.1, MT2492.SW; no longer CHRG.C, R17.1
- net N$9: now also DW01.OD, Q8.G1; no longer IC2.STAT, R17.2, R19.2
- net PMS_RX: now also J2.5; no longer X1-5.S
- net PMS_TX: now also J2.4; no longer X1-4.S
- net PWRKEY: now also C1.1; no longer D1.ANODE, GSM_RST.2
- net VBAT_EN: no longer R3.1
- net V_LIPO: now also BATT.NO1, BATT.NO2, C29.1, IP5306.BAT, L2.2, R19.2; no longer LIPO_SW.COM1, LIPO_SW.COM2
Other:
- note added: "GSM RESET"
- note removed: "CHARGING CIRCUIT"
- note removed: "LIPO BATTERY"
- note removed: "POWER KEY"
- moved on the sheet: C10, C11, C12, C13, C4, C9, D2, J3
