File: ESPS3_QuectelEC200U/V1/src/AQ_sensor_GSM.sch (EAGLE design)
At the start: 49 parts, among them IC2 MCP73831/OT, J1 F-1X03-SIP-100-32, SW1 PCM12SMTR, SW2 PCM12SMTR, U2 TEXAS_INSTRUMENTS_SN74HC125TE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, U3 TEXAS_INSTRUMENTS_LM1117IMP-3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, X1 53048-08, X2 SIMLOCK-C707_10M006_512_2, X4 50 Ohms

Commit message: V1 revised
Parts:
- removed CN1: (no value), AQ_sensor_GSM:JST_2PIN-SMT-RA
- removed D4: ON_SEMI_1N4148WSON_SEMI_1N4148WS_0_0, AQ_sensor_GSM:ON_SEMI_1N4148WSON_SEMI_1N4148WS_0_0
- removed NET: YELLOW, led:LEDCHIP-LED0603
- removed PWR: RED, led:LEDCHIP-LED0603
- removed R1, R6, R7: 470, rcl:R-EU_R0603
- removed RI: ORANGE, led:LEDCHIP-LED0603
- removed SW1, SW2: PCM12SMTR, AQ_sensor_GSM:PCM12SMTR
- removed TP1, TP2: TPB1,27, testpad:TPB1,27
- removed U2: TEXAS_INSTRUMENTS_SN74HC125TEXAS_INSTRUMENTS_SN74HC125_0_0, AQ_sensor_GSM:TEXAS_INSTRUMENTS_SN74HC125TEXAS_INSTRUMENTS_SN74HC125_0_0
- removed X2: SIMLOCK-C707_10M006_512_2, AQ_sensor_GSM:SIMLOCK-C707_10M006_512_2
- removed X4: 50 Ohms, AQ_sensor_GSM:SMACONNECTOR_EDGE_UFL
- added 10K, 51K, R12, R15, R21, R23, R3, R31, R34: 4.7K, rcl:R-EU_R0603
- added 3.7V_LIPO: 2828XX-2282837-2, Connector:2828XX-2282837-2
- added BT_ANT, GSMANTENNA2: (no value), SparkFun-Connectors:CONN_01
- added C12, C2: 470uf, T495X477K010ATE100:T495X477K010ATE100
- added C13, C18, C19, C20, C3, C7: 100nf, 06035C104K4T2A:06035C104K4T2A
- added C15, C16, C17: 33pF, rcl:C-EUC0603
- added C6: EEEFN1C471P, EEEFN1C471P:EEEFN1C471P
- added D5: ESD56151W04, 4.7V TVS Diode:1N4148WS_RR
- added EC200_GSM: EC200UCNAB-N05-SNNSA, EC200UCNAB-N05-SNNSA:EC200UCNAB-N05-SNNSA
- added ESP_RESET, GSM_RST: KMR621NGLFS, AQ_sensor_GSM:KMR621NGLFS
- added GPS, GSM: 1909763-1, 1909763-1:1909763-1
- added IC1: MIC29302WU, MIC29302WU:MIC29302WU
- added J3: PJ-002BH, PJ-002BH:PJ-002BH
- added LIPO_SW: TL2285EE, TL2285EE:TL2285EE
- added MICRO_SD1: TF-01A, TF-01A:TF-01A
- added M_RI, N_MODE, N_STAT, P_STAT: ORANGE, led:LEDCHIP-LED0603
- added Q1, Q2, Q3, Q4, Q5, Q6, Q7: MMBT2222, MMBT2222_:MMBT2222
- added R10, R13, R18, R22, R24, R32, R35, R8: 47K, rcl:R-EU_R0603
- added R11, R25, R28, R33, R36: 470R, rcl:R-EU_R0603
- added R2, R29, R30: 51K, rcl:R-EU_R0603
- added R26: 120K, rcl:R-EU_R0603
- added R27: 10K, rcl:R-EU_R0603
- added R9: 100k, rcl:R-EU_R0603
- added SIMCARD: 78646-3001, 78646-3001:78646-3001
- added U5: TXS0108EPWR, TXS0108EPWR:TXS0108EPWR
- S1: value KMR621NGLFS -> TL2285EE; device AQ_sensor_GSM:KMR621NGLFS -> TL2285EE:TL2285EE
- U1: value (none) -> LM7805S/NOPB; device AQ_sensor_GSM:GSM_SIM800L -> LM7805S_NOPB:LM7805S/NOPB
Connections:
- removed net 1.8V: D3.1_CATHODE, TP1.TP, U1.VSIM, X2.1
- removed net 2.8V: TP2.TP, U1.VEXT
- removed net GSM_RX: D4.ANODE, U1.UART_RXD
- removed net GSM_RX_O: D4.CATHODE, SV1.8
- removed net GSM_TX: U1.UART_TXD, U2B.2A
- removed net GSM_TX_5V: SV1.7, U2B.2Y
- removed net N$10: NET.A, R6.2
- removed net N$11: PWR.A, R7.2
- removed net N$14: R1.2, RI.A
- removed net NETSTAT_5V: R6.1, U2A.1Y
- removed net PWRSTAT_5V: R7.1, U2C.3Y
- removed net RI: U1.UART_RI, U2D.4A
- removed net RI_5V: RI.C, U2D.4Y
- removed net VIN: MICRO_USB.VUSB, SW1.2
- new net BP: 3.7V_LIPO.2, IC2.VBAT, LIPO_SW.NC1, LIPO_SW.NC2
- new net BT_ANT: BT_ANT.1, EC200_GSM.ANT_BT/WIFI_SCAN
- new net CP: C6.1, C7.2, D5.K, IC1.OUT, LIPO_SW.NO1, LIPO_SW.NO2, R11.2, R9.2
- new net GNSS_ANT: EC200_GSM.ANT_GNSS, GPS.SIG
- new net JACKP: J3.1, U1.IN
- new net MAIN_CTS: EC200_GSM.MAIN_CTS, U5.A3
- new net MAIN_DCD: EC200_GSM.MAIN_DCD, U5.A2
- new net MAIN_DTR: EC200_GSM.MAIN_DTR, U5.A5
- new net MAIN_RI: EC200_GSM.MAIN_RI, R34.1, U5.A1
- new net MAIN_RTS: EC200_GSM.MAIN_RTS, U5.A4
- new net MAIN_RXD: EC200_GSM.MAIN_RXD, U5.A7
- new net MAIN_TXD: EC200_GSM.MAIN_TXD, U5.A6
- new net MCU_CTS: U5.B3
- new net MCU_DCD: U5.B2
- new net MCU_DTR: SV2.11, U5.B5
- new net MCU_RI: U5.B1
- new net MCU_RTS: U5.B4
- new net MCU_RXD: SV1.8, U5.B6
- new net MCU_TXD: SV1.7, U5.B7
- new net N$1: Q2.B, R15.2, R18.2
- new net N$15: EC200_GSM.WLAN_PWR_EN
- new net N$16: EC200_GSM.WLAN_WAKE
- new net N$2: Q3.B, R21.2, R22.2
- new net N$22: Q5.B, R12.2, R13.2
- new net N$23: EC200_GSM.AP_READY
- new net N$26: Q4.B, R23.2, R24.2
- new net N$28: Q6.B, R31.2, R32.2
- new net N$29: Q4.C, R25.1
- new net N$30: N_MODE.C, R25.2
- new net N$31: R26.1, R27.2, U5.OE
- new net N$32: Q6.C, R33.1
- new net N$33: Q5.C, R28.1
- new net N$34: N_STAT.C, R28.2
- new net N$35: IC1.EN, Q1.C, R2.1
- new net N$36: Q1.B, R3.2
- new net N$37: Q1.E, R8.2
- new net N$38: IC1.ADJ, R10.2, R9.1
- new net N$39: P_STAT.C, R33.2
- new net N$40: R30.1, U5.A8
- new net N$41: R29.1, U5.B8
- new net N$42: Q7.B, R34.2, R35.2
- new net N$43: Q7.C, R36.1
- new net N$44: M_RI.C, R36.2
- new net N$5: EC200_GSM.USIM2_VDD
- new net N$7: EC200_GSM.BT_EN
- new net N$8: EC200_GSM.WLAN_EN
- new net NET_MODE: EC200_GSM.NET_MODE, R23.1
- new net PWRKEY_0: R21.1, SV1.15
- new net TF-CLK: MICRO_SD1.CLK, SV2.7
- new net TF-CS: MICRO_SD1.CD/DAT3, SV2.9
- new net TF-MISO: MICRO_SD1.DAT0, SV2.8
- new net TF-MOSI: MICRO_SD1.CMD, SV2.10
- new net USBP: MICRO_USB.VUSB, S1.COM1, S1.COM2
- new net USIM_DET: 51K.1, D3.5_CATHODE, EC200_GSM.USIM_DET
- new net USIM_GND: C18.1, EC200_GSM.USIM_GND
- new net USIM_VDD: 10K.2, C18.2, D3.1_CATHODE, EC200_GSM.USIM_VDD, SIMCARD.VCC
- new net VBAT_EN: R3.1, SV2.12
- new net VDD_EXT: 51K.2, C19.2, EC200_GSM.VDD_EXT, R27.1, U5.VCCA
- net +3V3: now also C20.2, MICRO_SD1.VDD, SV1.10, U5.VCCB
- net +5V: now also C2.1, C3.2, IC1.VIN, R2.2, S1.NO1, S1.NO2, U1.OUT; no longer R1.1, SW1.1, U2E.VCC
- net ESP_RST: now also ESP_RESET.2; no longer SW2.2
- net GND: now also 3.7V_LIPO.1, C12.2, C13.1, C15.2, C16.2, C17.2, C19.1, C2.2, C20.1, C3.1, C6.2, C7.1, D5.A, EC200_GSM.GND, ESP_RESET.1, GPS.GND, GSM.GND, GSM_RST.1, IC1.GND, J3.2, J3.3, MICRO_SD1.SHIELD, MICRO_SD1.VSS, Q2.E, Q3.E, Q4.E, Q5.E, Q6.E, Q7.E, R10.1, R11.1, R13.1, R18.1, R22.1, R24.1, R26.2, R29.2, R30.2, R32.1, R35.1, R8.1, SIMCARD.GND, SV1.9, U5.GND; no longer CN1.1, NET.C, PWR.C, S1.1, SW1.SHIELD, SW2.1, SW2.SHIELD, U2A.1_!OE!, U2B.4_!OE!, U2C.2_!OE!, U2D.3_!OE!, U2E.GND, X2.4, X4.GND1, X4.GND2, X4.GND3, X4.GND4
- net GSM_ANT: now also EC200_GSM.ANT_MAIN, GSM.SIG, GSMANTENNA2.1; no longer U1.ANT, X4.ANT
- net GSM_RST: now also EC200_GSM.!RESET, Q2.C; no longer U1.RESET
- net GSM_RST_O: now also R15.1
- net NETSTAT: now also EC200_GSM.NET_STATUS, R12.1; no longer U1.NETLIGHT, U2A.1A
- net PWRKEY: now also EC200_GSM.PWRKEY, GSM_RST.2, Q3.C; no longer S1.2, U1.PWRKEY
- net PWRSTAT: now also EC200_GSM.STATUS, R31.1; no longer U1.STATUS, U2C.3A
- net SIMCLK: now also C16.1, EC200_GSM.USIM_CLK, SIMCARD.CLK; no longer U1.SIM_CLK, X2.3
- net SIMDATA: now also 10K.1, C15.1, EC200_GSM.USIM_DATA, SIMCARD.I/O; no longer U1.SIM_DATA, X2.6
- net SIMRST: now also C17.1, EC200_GSM.USIM_RST, SIMCARD.RST; no longer U1.SIM_RST, X2.2
- net VRTC: no longer U1.VRTC
- net V_LIPO: now also C12.1, C13.2, EC200_GSM.VBAT_BB, EC200_GSM.VBAT_RF, LIPO_SW.COM1, LIPO_SW.COM2, M_RI.A, N_MODE.A, N_STAT.A, P_STAT.A; no longer CN1.2, IC2.VBAT, U1.VBAT
Other:
- note added: "GNSS ANTENNA"
- note removed: "LEVEL SHIFTER"
- note removed: "SIM800H"
- note removed: "STATUS LEDS"
- note removed: "TEST PADS"
